File: MCU/mcu/output_clamp_and_ADC_Interface.kicad_sch (KiCad schematic)
At the start: 3 parts, among them U3 ADS8688

Commit message: worked on unit 5
Parts:
- removed D2: ESD5Zxx, Diode_SMD:D_SOD-523, symbol Diode:ESD5Zxx
- removed R9: R, symbol Device:R
- added D8: ESD5Z3.3TiG, symbol Device:D_Schottky
- added R12: 100, symbol Device:R
Connections:
- net In: now also R12.1
- net at U3.16 (AIN_0P): now also D8.1 (K), R12.2
- new net GND: D8.2 (A)
Changed lines of the file:
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@@
 	(generator_version "10.0")
 	(paper "A4")
+	(junction
+		(at 143.51 73.66)
+		(diameter 0)
+		(color 0 0 0 0)
+	)
+	(wire
+		(pts
+			(xy 157.48 72.39) (xy 157.48 96.52)
+		)
+		(stroke
+			(width 0)
+			(type default)
+		)
+	)
+	(wire
+		(pts
+			(xy 143.51 45.72) (xy 143.51 73.66)
+		)
+		(stroke
+			(width 0)
+			(type default)
+		)
+	)
+	(wire
+		(pts
+			(xy 187.96 45.72) (xy 143.51 45.72)
+		)
+		(stroke
+			(width 0)
+			(type default)
+		)
+	)
+	(wire
+		(pts
+			(xy 157.48 96.52) (xy 158.75 96.52)
+		)
+		(stroke
+			(width 0)
+			(type default)
+		)
+	)
+	(wire
+		(pts
+			(xy 118.11 78.74) (xy 118.11 73.66)
+		)
+		(stroke
+			(width 0)
+			(type default)
+		)
+	)
+	(wire
+		(pts
+			(xy 125.73 73.66) (xy 143.51 73.66)
+		)
+		(stroke
+			(width 0)
+			(type default)
+		)
+	)
+	(wire
+		(pts
+			(xy 146.05 73.66) (xy 146.05 72.39)
+		)
+		(stroke
+			(width 0)
+			(type default)
+		)
+	)
+	(wire
+		(pts
+			(xy 39.37 78.74) (xy 118.11 78.74)
+		)
+		(stroke
+			(width 0)
+			(type default)
+		)
+	)
+	(wire
+		(pts
+			(xy 143.51 73.66) (xy 146.05 73.66)
+		)
+		(stroke
+			(width 0)
+			(type default)
+		)
+	)
+	(wire
+		(pts
+			(xy 153.67 72.39) (xy 157.48 72.39)
+		)
+		(stroke
+			(width 0)
+			(type default)
+		)
+	)
 	(hierarchical_label "In"
-		(shape output)
+		(shape input)
 		(at 39.37 78.74 180)
 		(effects
@@
 	)
 	(symbol
-		(lib_id "Device:R")
-		(at 64.77 48.26 90)
+		(lib_id "Device:D_Schottky")
+		(at 149.86 72.39 0)
 		(unit 1)
 		(body_style 1)
@@
 		(dnp no)
 		(fields_autoplaced yes)
-		(property "Reference" "R9"
-			(at 64.77 41.91 90)
-			(show_name no)
-			(do_not_autoplace no)
-			(effects
-				(font
-					(size 1.27 1.27)
-				)
-			)
-		)
-		(property "Value" "R"
-			(at 64.77 44.45 90)
+		(property "Reference" "D8"
+			(at 149.5425 66.04 0)
+			(show_name no)
+			(do_not_autoplace no)
+			(effects
+				(font
+					(size 1.27 1.27)
+				)
+			)
+		)
+		(property "Value" "ESD5Z3.3TiG"
+			(at 149.5425 68.58 0)
 			(show_name no)
 			(do_not_autoplace no)
@@
 		)
 		(property "Footprint" ""
-			(at 64.77 50.038 90)
+			(at 149.86 72.39 0)
 			(hide yes)
 			(show_name no)
@@
 		)
 		(property "Datasheet" ""
-			(at 64.77 48.26 0)
-			(hide yes)
-			(show_name no)
-			(do_not_autoplace no)
-			(effects
-				(font
-					(size 1.27 1.27)
-				)
-			)
-		)
-		(property "Description" "Resistor"
-			(at 64.77 48.26 0)
-			(hide yes)
-			(show_name no)
-			(do_not_autoplace no)
-			(effects
-				(font
-					(size 1.27 1.27)
-				)
-			)
+			(at 149.86 72.39 0)
+			(hide yes)
+			(show_name no)
+			(do_not_autoplace no)
+			(effects
+				(font
+					(size 1.27 1.27)
+				)
+			)
+		)
+		(property "Description" "Schottky diode"
+			(at 149.86 72.39 0)
+			(hide yes)
+			(show_name no)
+			(do_not_autoplace no)
+			(effects
+				(font
+					(size 1.27 1.27)
+				)
+			)
+		)
+		(pin "1"
 		)
 		(pin "2"
-		)
-		(pin "1"
 		)
 		(instances
 			(project "mcu"
 				(path "/a05656f2-56dd-4122-820d-a34d3928231b/7e909fd8-f3c4-41fd-9605-74d0338eac58"
-					(reference "R9")
+					(reference "D8")
+					(unit 1)
+				)
+			)
+		)
+	)
+	(symbol
+		(lib_id "power:GND")
+		(at 158.75 96.52 0)
+		(unit 1)
+		(body_style 1)
+		(exclude_from_sim no)
+		(in_bom yes)
+		(on_board yes)
+		(in_pos_files yes)
+		(dnp no)
+		(fields_autoplaced yes)
+		(property "Reference" "#PWR021"
+			(at 158.75 102.87 0)
+			(hide yes)
+			(show_name no)
+			(do_not_autoplace no)
+			(effects
+				(font
+					(size 1.27 1.27)
+				)
+			)
+		)
+		(property "Value" "GND"
+			(at 158.75 101.6 0)
+			(show_name no)
+			(do_not_autoplace no)
+			(effects
+				(font
+					(size 1.27 1.27)
+				)
+			)
+		)
+		(property "Footprint" ""
+			(at 158.75 96.52 0)
+			(hide yes)
+			(show_name no)
+			(do_not_autoplace no)
+			(effects
+				(font
+					(size 1.27 1.27)
+				)
+			)
+		)
+		(property "Datasheet" ""
+			(at 158.75 96.52 0)
+			(hide yes)
+			(show_name no)
+			(do_not_autoplace no)
+			(effects
+				(font
+					(size 1.27 1.27)
+				)
+			)
+		)
+		(property "Description" "Power symbol creates a global label with name \"GND\" , ground"
+			(at 158.75 96.52 0)
+			(hide yes)
+			(show_name no)
+			(do_not_autoplace no)
+			(effects
+				(font
+					(size 1.27 1.27)
+				)
+			)
+		)
+		(pin "1"
+		)
+		(instances
+			(project "mcu"
+				(path "/a05656f2-56dd-4122-820d-a34d3928231b/7e909fd8-f3c4-41fd-9605-74d0338eac58"
+					(reference "#PWR021")
 					(unit 1)
 				)
@@
 	)
 	(symbol
-		(lib_id "Diode:ESD5Zxx")
-		(at 113.03 49.53 0)
+		(lib_id "Device:R")
+		(at 121.92 73.66 90)
 		(unit 1)
 		(body_style 1)
@@
 		(dnp no)
 		(fields_autoplaced yes)
-		(property "Reference" "D2"
-			(at 113.03 43.18 0)
-			(show_name no)
-			(do_not_autoplace no)
-			(effects
-				(font
-					(size 1.27 1.27)
-				)
-			)
-		)
-		(property "Value" "ESD5Zxx"
-			(at 113.03 45.72 0)
-			(show_name no)
-			(do_not_autoplace no)
-			(effects
-				(font
-					(size 1.27 1.27)
-				)
-			)
-		)
-		(property "Footprint" "Diode_SMD:D_SOD-523"
-			(at 113.03 53.975 0)
-			(hide yes)
-			(show_name no)
-			(do_not_autoplace no)
-			(effects
-				(font
-					(size 1.27 1.27)
-				)
-			)
-		)
-		(property "Datasheet" "https://www.onsemi.com/pdf/datasheet/esd5z2.5t1-d.pdf"
-			(at 113.03 49.53 0)
-			(hide yes)
-			(show_name no)
-			(do_not_autoplace no)
-			(effects
-				(font
-					(size 1.27 1.27)
-				)
-			)
-		)
-		(property "Description" "ESD Protection Diode, SOD-523"
-			(at 113.03 49.53 0)
-			(hide yes)
-			(show_name no)
-			(do_not_autoplace no)
-			(effects
-				(font
-					(size 1.27 1.27)
-				)
-			)
+		(property "Reference" "R12"
+			(at 121.92 67.31 90)
+			(show_name no)
+			(do_not_autoplace no)
+			(effects
+				(font
+					(size 1.27 1.27)
+				)
+			)
+		)
+		(property "Value" "100"
+			(at 121.92 69.85 90)
+			(show_name no)
+			(do_not_autoplace no)
+			(effects
+				(font
+					(size 1.27 1.27)
+				)
+			)
+		)
+		(property "Footprint" ""
+			(at 121.92 75.438 90)
+			(hide yes)
+			(show_name no)
+			(do_not_autoplace no)
+			(effects
+				(font
+					(size 1.27 1.27)
+				)
+			)
+		)
+		(property "Datasheet" ""
+			(at 121.92 73.66 0)
+			(hide yes)
+			(show_name no)
+			(do_not_autoplace no)
+			(effects
+				(font
+					(size 1.27 1.27)
+				)
+			)
+		)
+		(property "Description" "Resistor"
+			(at 121.92 73.66 0)
+			(hide yes)
+			(show_name no)
+			(do_not_autoplace no)
+			(effects
+				(font
+					(size 1.27 1.27)
+				)
+			)
+		)
+		(pin "2"
 		)
 		(pin "1"
-		)
-		(pin "2"
 		)
 		(instances
 			(project "mcu"
 				(path "/a05656f2-56dd-4122-820d-a34d3928231b/7e909fd8-f3c4-41fd-9605-74d0338eac58"
-					(reference "D2")
+					(reference "R12")
 					(unit 1)
 				)

Commit message: working on 5
Parts:
- added C12: 1u, symbol Device:C
- added C13: 10u, symbol Device:C
- added C14: 4.7u, symbol Device:C
- added C16: 0.1u, symbol Device:C
- added R13, R9: 10k, symbol Device:R
- added U4: STM32F401CCUx, Package_DFN_QFN:QFN-48-1EP_7x7mm_P0.5mm_EP5.6x5.6mm, symbol MCU_ST_STM32F4:STM32F401CCUx
- D8: footprint (none) -> D_SOD-523
- R12: footprint (none) -> R_0603_1608Metric
Connections:
- net GND: now also U3.28 (AGND), U3.29 (AGND), U3.31 (AGND), U3.32 (AGND), U3.33 (DGND), U3.6 (REFGND), U3.8 (AGND), C12.2, C13.2, C14.2, C16.2, R9.2, U4.23 (VSS), U4.35 (VSS), U4.47 (VSS), U4.49 (VSS), U4.8 (VSSA)
- net at U3.1 (SDI): now also U4.17 (PA7)
- net at U3.2 (~{RST/PD}): now also U4.13 (PA3)
- net +5V: now reaches U3.30 (AVDD)
- net +5V: now also U3.9 (AVDD)
- net +3.3V: now reaches U3.34 (DVDD)
- net +3.3V: now also R13.1, U4.1 (VBAT), U4.24 (VDD), U4.36 (VDD), U4.48 (VDD)
- net at U3.36 (SDO): now also U4.16 (PA6)
- net at U3.37 (SCLK): now also U4.15 (PA5)
- net at U3.38 (~{CS}): now also U4.14 (PA4)
- net at U3.5 (REFIO): now also C13.1
- net at U3.7 (REFCAP): now also C12.1
- new net: C14.1, U4.22 (VCAP1)
- new net: R9.1, U4.44 (BOOT0)
- new net: C16.1, R13.2, U4.7 (NRST)
- no-connect marks 0 -> 51

Commit message: added footprints
Parts:
- C12, C13, C14, C16: footprint (none) -> Capacitor_SMD:C_0805_2012Metric
- R13, R9: footprint (none) -> Resistor_SMD:R_0805_2012Metric
Changed lines of the file:
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@@
 			)
 		)
-		(property "Footprint" ""
+		(property "Footprint" "Capacitor_SMD:C_0805_2012Metric"
 			(at 234.6452 120.65 0)
 			(hide yes)
@@
 			)
 		)
-		(property "Footprint" ""
+		(property "Footprint" "Resistor_SMD:R_0805_2012Metric"
 			(at 226.822 67.31 90)
 			(hide yes)
@@
 			)
 		)
-		(property "Footprint" ""
+		(property "Footprint" "Capacitor_SMD:C_0805_2012Metric"
 			(at 223.2152 71.12 0)
 			(hide yes)
@@
 			)
 		)
-		(property "Footprint" ""
+		(property "Footprint" "Resistor_SMD:R_0805_2012Metric"
 			(at 213.36 36.068 90)
 			(hide yes)
@@
 			)
 		)
-		(property "Footprint" ""
+		(property "Footprint" "Capacitor_SMD:C_0805_2012Metric"
 			(at 220.6752 77.47 0)
 			(hide yes)
@@
 			)
 		)
-		(property "Footprint" ""
+		(property "Footprint" "Capacitor_SMD:C_0805_2012Metric"
 			(at 227.0252 85.09 0)
 			(hide yes)
