File: MCU/mcu/anti_aliasing.kicad_sch (KiCad schematic)
At the start: 7 parts, among them U2 MCP6002-xMS

Commit message: added footprints
Parts:
- C4, C6, C7: footprint (none) -> Capacitor_SMD:C_0805_2012Metric
- R5, R6, R8: footprint (none) -> Resistor_SMD:R_0805_2012Metric
- U2: footprint (none) -> Package_SO:MSOP-8_3x3mm_P0.65mm
Changed lines of the file:
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@@
 			)
 		)
-		(property "Footprint" ""
+		(property "Footprint" "Resistor_SMD:R_0805_2012Metric"
 			(at 59.69 64.008 90)
 			(hide yes)
@@
 			)
 		)
-		(property "Footprint" ""
+		(property "Footprint" "Capacitor_SMD:C_0805_2012Metric"
 			(at 68.8848 39.37 0)
 			(hide yes)
@@
 			)
 		)
-		(property "Footprint" ""
+		(property "Footprint" "Package_SO:MSOP-8_3x3mm_P0.65mm"
 			(at 146.05 52.07 0)
 			(hide yes)
@@
 			)
 		)
-		(property "Footprint" ""
+		(property "Footprint" "Package_SO:MSOP-8_3x3mm_P0.65mm"
 			(at 205.74 52.07 0)
 			(hide yes)
@@
 			)
 		)
-		(property "Footprint" ""
+		(property "Footprint" "Package_SO:MSOP-8_3x3mm_P0.65mm"
 			(at 241.3 132.08 0)
 			(hide yes)
@@
 			)
 		)
-		(property "Footprint" ""
+		(property "Footprint" "Resistor_SMD:R_0805_2012Metric"
 			(at 175.26 56.388 90)
 			(hide yes)
@@
 			)
 		)
-		(property "Footprint" ""
+		(property "Footprint" "Capacitor_SMD:C_0805_2012Metric"
 			(at 190.5 87.9348 0)
 			(hide yes)
@@
 			)
 		)
-		(property "Footprint" ""
+		(property "Footprint" "Capacitor_SMD:C_0805_2012Metric"
 			(at 107.95 91.1352 0)
 			(hide yes)
@@
 			)
 		)
-		(property "Footprint" ""
+		(property "Footprint" "Resistor_SMD:R_0805_2012Metric"
 			(at 81.28 64.008 90)
 			(hide yes)

Commit message: cleaned 3,4
Parts:
- removed C7: C, Capacitor_SMD:C_0805_2012Metric, symbol Device:C
- removed R8: 10k, Resistor_SMD:R_0805_2012Metric, symbol Device:R
- added C15: 130p, Capacitor_SMD:C_0805_2012Metric, symbol Device:C
- C6: value C -> 510p
Connections:
- net GND: now also U2.2 (-), C15.1; no longer U2.3 (+), U2.5 (+)
- net Out: now also U2.6 (-)
- net at C4.1, R5.2, R6.1: no longer C6.2
- net at C6.1, U2.1: now also U2.5 (+), C15.2
- net at R6.2: now also C6.2, U2.3 (+); no longer U2.2 (-)
