File: MCU/mcu/anti_aliasing.kicad_sch (KiCad schematic)
At the start: 6 parts, among them U2 MCP6002-xMS

Commit message: trying simulation
Other:
- note added: ".tran 10m 100m"
Changed lines of the file:
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@@
 	(generator_version "10.0")
 	(paper "A4")
+	(text ".tran 10m 100m"
+		(exclude_from_sim no)
+		(at 71.374 111.76 0)
+		(effects
+			(font
+				(size 1.27 1.27)
+			)
+		)
+	)
 	(junction
 		(at 129.54 93.98)
