File: MCU/mcu/anti_aliasing.kicad_sch (KiCad schematic)
At the start: 6 parts, among them U2 MCP6002-xMS

Commit message: changed
Parts:
- removed C15: 130p, Capacitor_SMD:C_0805_2012Metric, symbol Device:C
Connections:
- net GND: now also C6.1; no longer C4.2
- net at U2.1, U2.5 (+): now also C4.2; no longer C6.1
Changed lines of the file:
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@@
-	)
-	(junction
-		(at 129.54 93.98)
-		(diameter 0)
-		(color 0 0 0 0)
 	)
 	(junction
@@
 	)
 	(junction
-		(at 153.67 52.07)
+		(at 168.91 52.07)
 		(diameter 0)
 		(color 0 0 0 0)
 	)
 	(junction
-		(at 165.1 52.07)
+		(at 139.7 34.29)
 		(diameter 0)
 		(color 0 0 0 0)
@@
 	(wire
 		(pts
-			(xy 137.16 34.29) (xy 165.1 34.29)
-		)
-		(stroke
-			(width 0)
-			(type default)
-		)
-	)
-	(wire
-		(pts
-			(xy 153.67 52.07) (xy 165.1 52.07)
-		)
-		(stroke
-			(width 0)
-			(type default)
-		)
-	)
-	(wire
-		(pts
-			(xy 90.17 27.94) (xy 90.17 40.64)
-		)
-		(stroke
-			(width 0)
-			(type default)
-		)
-	)
-	(wire
-		(pts
-			(xy 165.1 34.29) (xy 165.1 52.07)
-		)
-		(stroke
-			(width 0)
-			(type default)
-		)
-	)
-	(wire
-		(pts
-			(xy 153.67 52.07) (xy 153.67 93.98)
+			(xy 139.7 34.29) (xy 139.7 35.56)
+		)
+		(stroke
+			(width 0)
+			(type default)
+		)
+	)
+	(wire
+		(pts
+			(xy 114.3 27.94) (xy 114.3 16.51)
 		)
 		(stroke
@@
 	(wire
 		(pts
-			(xy 165.1 52.07) (xy 171.45 52.07)
+			(xy 153.67 52.07) (xy 168.91 52.07)
 		)
 		(stroke
@@
 	(wire
 		(pts
-			(xy 137.16 93.98) (xy 153.67 93.98)
+			(xy 114.3 16.51) (xy 168.91 16.51)
+		)
+		(stroke
+			(width 0)
+			(type default)
+		)
+	)
+	(wire
+		(pts
+			(xy 168.91 52.07) (xy 171.45 52.07)
 		)
 		(stroke
@@
 	(wire
 		(pts
+			(xy 139.7 34.29) (xy 152.4 34.29)
+		)
+		(stroke
+			(width 0)
+			(type default)
+		)
+	)
+	(wire
+		(pts
+			(xy 137.16 34.29) (xy 139.7 34.29)
+		)
+		(stroke
+			(width 0)
+			(type default)
+		)
+	)
+	(wire
+		(pts
 			(xy 63.5 62.23) (xy 69.85 62.23)
 		)
@@
 	(wire
 		(pts
+			(xy 168.91 16.51) (xy 168.91 52.07)
+		)
+		(stroke
+			(width 0)
+			(type default)
+		)
+	)
+	(wire
+		(pts
 			(xy 129.54 49.53) (xy 138.43 49.53)
 		)
@@
 	(wire
 		(pts
-			(xy 69.85 27.94) (xy 90.17 27.94)
+			(xy 69.85 27.94) (xy 114.3 27.94)
 		)
 		(stroke
@@
 		(instances
 			(project "mcu"
-				(path "/a05656f2-56dd-4122-820d-a34d3928231b/d9d41d52-a750-4c10-a354-fe076c41d7d7"
+				(path "/a05656f2-56dd-4122-820d-a34d3928231b/090f5bd0-76cd-4f87-9c27-4571509190da"
 					(reference "R5")
 					(unit 1)
@@
 		(instances
 			(project "mcu"
-				(path "/a05656f2-56dd-4122-820d-a34d3928231b/d9d41d52-a750-4c10-a354-fe076c41d7d7"
+				(path "/a05656f2-56dd-4122-820d-a34d3928231b/090f5bd0-76cd-4f87-9c27-4571509190da"
 					(reference "C4")
 					(unit 1)
@@
 		(instances
 			(project "mcu"
-				(path "/a05656f2-56dd-4122-820d-a34d3928231b/d9d41d52-a750-4c10-a354-fe076c41d7d7"
+				(path "/a05656f2-56dd-4122-820d-a34d3928231b/090f5bd0-76cd-4f87-9c27-4571509190da"
 					(reference "#PWR010")
 					(unit 1)
@@
 			)
 		)
-		(property "Sim.Library" "spice/MCP6001_MM_G/MCP6002.txt"
+		(property "Sim.Library" "spice\\MCP6001_MM_G\\MCP6002.txt"
 			(at 146.05 52.07 0)
 			(hide yes)
@@
 		(instances
 			(project "mcu"
-				(path "/a05656f2-56dd-4122-820d-a34d3928231b/d9d41d52-a750-4c10-a354-fe076c41d7d7"
+				(path "/a05656f2-56dd-4122-820d-a34d3928231b/090f5bd0-76cd-4f87-9c27-4571509190da"
 					(reference "U2")
 					(unit 1)
@@
 			)
 		)
-		(property "Sim.Library" "spice/MCP6001_MM_G/MCP6002.txt"
+		(property "Sim.Library" "spice\\MCP6001_MM_G\\MCP6002.txt"
 			(at 205.74 52.07 0)
 			(hide yes)
@@
 		(instances
 			(project "mcu"
-				(path "/a05656f2-56dd-4122-820d-a34d3928231b/d9d41d52-a750-4c10-a354-fe076c41d7d7"
+				(path "/a05656f2-56dd-4122-820d-a34d3928231b/090f5bd0-76cd-4f87-9c27-4571509190da"
 					(reference "U2")
 					(unit 2)
@@
 		(instances
 			(project "mcu"
-				(path "/a05656f2-56dd-4122-820d-a34d3928231b/d9d41d52-a750-4c10-a354-fe076c41d7d7"
+				(path "/a05656f2-56dd-4122-820d-a34d3928231b/090f5bd0-76cd-4f87-9c27-4571509190da"
 					(reference "#PWR012")
 					(unit 1)
@@
 			)
 		)
-		(property "Sim.Library" "spice/MCP6001_MM_G/MCP6002.txt"
+		(property "Sim.Library" "spice\\MCP6001_MM_G\\MCP6002.txt"
 			(at 241.3 132.08 0)
 			(hide yes)
@@
 		(instances
 			(project "mcu"
-				(path "/a05656f2-56dd-4122-820d-a34d3928231b/d9d41d52-a750-4c10-a354-fe076c41d7d7"
+				(path "/a05656f2-56dd-4122-820d-a34d3928231b/090f5bd0-76cd-4f87-9c27-4571509190da"
 					(reference "U2")
 					(unit 3)
@@
 		(instances
 			(project "mcu"
-				(path "/a05656f2-56dd-4122-820d-a34d3928231b/d9d41d52-a750-4c10-a354-fe076c41d7d7"
+				(path "/a05656f2-56dd-4122-820d-a34d3928231b/090f5bd0-76cd-4f87-9c27-4571509190da"
 					(reference "C6")
-					(unit 1)
-				)
-			)
-		)
-	)
-	(symbol
-		(lib_id "power:GND")
-		(at 90.17 40.64 0)
-		(unit 1)
-		(body_style 1)
-		(exclude_from_sim no)
-		(in_bom yes)
-		(on_board yes)
-		(in_pos_files yes)
-		(dnp no)
-		(fields_autoplaced yes)
-		(property "Reference" "#PWR013"
-			(at 90.17 46.99 0)
-			(hide yes)
-			(show_name no)
-			(do_not_autoplace no)
-			(effects
-				(font
-					(size 1.27 1.27)
-				)
-			)
-		)
-		(property "Value" "GND"
-			(at 90.17 45.72 0)
-			(show_name no)
-			(do_not_autoplace no)
-			(effects
-				(font
-					(size 1.27 1.27)
-				)
-			)
-		)
-		(property "Footprint" ""
-			(at 90.17 40.64 0)
-			(hide yes)
-			(show_name no)
-			(do_not_autoplace no)
-			(effects
-				(font
-					(size 1.27 1.27)
-				)
-			)
-		)
-		(property "Datasheet" ""
-			(at 90.17 40.64 0)
-			(hide yes)
-			(show_name no)
-			(do_not_autoplace no)
-			(effects
-				(font
-					(size 1.27 1.27)
-				)
-			)
-		)
-		(property "Description" "Power symbol creates a global label with name \"GND\" , ground"
-			(at 90.17 40.64 0)
-			(hide yes)
-			(show_name no)
-			(do_not_autoplace no)
-			(effects
-				(font
-					(size 1.27 1.27)
-				)
-			)
-		)
-		(pin "1"
-		)
-		(instances
-			(project "mcu"
-				(path "/a05656f2-56dd-4122-820d-a34d3928231b/d9d41d52-a750-4c10-a354-fe076c41d7d7"
-					(reference "#PWR013")
 					(unit 1)
 				)
@@
 		(instances
 			(project "mcu"
-				(path "/a05656f2-56dd-4122-820d-a34d3928231b/d9d41d52-a750-4c10-a354-fe076c41d7d7"
+				(path "/a05656f2-56dd-4122-820d-a34d3928231b/090f5bd0-76cd-4f87-9c27-4571509190da"
 					(reference "#PWR011")
+					(unit 1)
+				)
+			)
+		)
+	)
+	(symbol
+		(lib_id "power:GND")
+		(at 152.4 34.29 0)
+		(unit 1)
+		(body_style 1)
+		(exclude_from_sim no)
+		(in_bom yes)
+		(on_board yes)
+		(in_pos_files yes)
+		(dnp no)
+		(fields_autoplaced yes)
+		(property "Reference" "#PWR013"
+			(at 152.4 40.64 0)
+			(hide yes)
+			(show_name no)
+			(do_not_autoplace no)
+			(effects
+				(font
+					(size 1.27 1.27)
+				)
+			)
+		)
+		(property "Value" "GND"
+			(at 152.4 39.37 0)
+			(show_name no)
+			(do_not_autoplace no)
+			(effects
+				(font
+					(size 1.27 1.27)
+				)
+			)
+		)
+		(property "Footprint" ""
+			(at 152.4 34.29 0)
+			(hide yes)
+			(show_name no)
+			(do_not_autoplace no)
+			(effects
+				(font
+					(size 1.27 1.27)
+				)
+			)
+		)
+		(property "Datasheet" ""
+			(at 152.4 34.29 0)
+			(hide yes)
+			(show_name no)
+			(do_not_autoplace no)
+			(effects
+				(font
+					(size 1.27 1.27)
+				)
+			)
+		)
+		(property "Description" "Power symbol creates a global label with name \"GND\" , ground"
+			(at 152.4 34.29 0)
+			(hide yes)
+			(show_name no)
+			(do_not_autoplace no)
+			(effects
+				(font
+					(size 1.27 1.27)
+				)
+			)
+		)
+		(pin "1"
+		)
+		(instances
+			(project "mcu"
+				(path "/a05656f2-56dd-4122-820d-a34d3928231b/090f5bd0-76cd-4f87-9c27-4571509190da"
+					(reference "#PWR013")
 					(unit 1)
 				)
@@
 		(instances
 			(project "mcu"
-				(path "/a05656f2-56dd-4122-820d-a34d3928231b/d9d41d52-a750-4c10-a354-fe076c41d7d7"
+				(path "/a05656f2-56dd-4122-820d-a34d3928231b/090f5bd0-76cd-4f87-9c27-4571509190da"
 					(reference "R6")
 					(unit 1)
 				)
-			)
-		)
-	)
-	(symbol
-		(lib_id "Device:C")
-		(at 133.35 93.98 90)
-		(unit 1)
-		(body_style 1)
-		(exclude_from_sim no)
-		(in_bom yes)
-		(on_board yes)
-		(in_pos_files yes)
-		(dnp no)
-		(fields_autoplaced yes)
-		(property "Reference" "C15"
-			(at 133.35 86.36 90)
-			(show_name no)
-			(do_not_autoplace no)
-			(effects
-				(font
-					(size 1.27 1.27)
-				)
-			)
-		)
-		(property "Value" "130p"
-			(at 133.35 88.9 90)
-			(show_name no)
-			(do_not_autoplace no)
-			(effects
-				(font
-					(size 1.27 1.27)
-				)
-			)
-		)
-		(property "Footprint" "Capacitor_SMD:C_0805_2012Metric"
-			(at 137.16 93.0148 0)
-			(hide yes)
-			(show_name no)
-			(do_not_autoplace no)
-			(effects
-				(font
-					(size 1.27 1.27)
-				)
-			)
-		)
-		(property "Datasheet" ""
-			(at 133.35 93.98 0)
-			(hide yes)
-			(show_name no)
-			(do_not_autoplace no)
-			(effects
-				(font
-					(size 1.27 1.27)
-				)
-			)
-		)
-		(property "Description" "Unpolarized capacitor"
-			(at 133.35 93.98 0)
-			(hide yes)
-			(show_name no)
-			(do_not_autoplace no)
-			(effects
-				(font
-					(size 1.27 1.27)
-				)
-			)
-		)
-		(pin "2"
-		)
-		(pin "1"
-		)
-		(instances
-			(project "mcu"
-				(path "/a05656f2-56dd-4122-820d-a34d3928231b/d9d41d52-a750-4c10-a354-fe076c41d7d7"
-					(reference "C15")
-					(unit 1)
-				)

Commit message: yy
Parts:
- added C1: 1n, symbol Device:C
- added C2: 150p, symbol Device:C
- added R2, R3: 20k, symbol Device:R
- added V3, V4: VSIN, symbol Simulation_SPICE:VSIN
- C4: value 0.27n -> 430pf
- C6: value 510p -> 360p
Connections:
- net GND: now also C2.2, V3.2; no longer U2.2 (-)
- net Out: now also C1.1
- net at C4.2, U2.1: now also U2.2 (-), R3.1; no longer U2.5 (+)
- net In: no longer names the net of R5.1
- net In: now also V4.1
- new net: C2.1, R2.2, U2.5 (+)
- new net: V3.1, V4.2
- new net: C1.2, R2.1, R3.2
Other:
- note added: ".ac dec 20 1 1Meg"
- note removed: ".tran 10m 100m"
- moved on the sheet: U2B
