File: MCU/mcu/instrumentation_amplifier.kicad_sch (KiCad schematic)
At the start: 13 parts, among them U1 INA128

Commit message: added footprints
Parts:
- C10, C11, C5, C8, C9: footprint (none) -> Capacitor_SMD:C_0805_2012Metric
- R10, R11, R7: footprint (none) -> Resistor_SMD:R_0805_2012Metric
- U1: footprint (none) -> Package_SO:SOIC-8_3.9x4.9mm_P1.27mm
Changed lines of the file:
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@@
 			)
 		)
-		(property "Footprint" ""
+		(property "Footprint" "Resistor_SMD:R_0805_2012Metric"
 			(at 34.29 53.848 90)
 			(hide yes)
@@
 			)
 		)
-		(property "Footprint" ""
+		(property "Footprint" "Capacitor_SMD:C_0805_2012Metric"
 			(at 88.5952 67.31 0)
 			(hide yes)
@@
 			)
 		)
-		(property "Footprint" ""
+		(property "Footprint" "Capacitor_SMD:C_0805_2012Metric"
 			(at 42.2148 41.91 0)
 			(hide yes)
@@
 			)
 		)
-		(property "Footprint" ""
+		(property "Footprint" "Capacitor_SMD:C_0805_2012Metric"
 			(at 79.7052 67.31 0)
 			(hide yes)
@@
 			)
 		)
-		(property "Footprint" ""
+		(property "Footprint" "Capacitor_SMD:C_0805_2012Metric"
 			(at 45.4152 72.39 0)
 			(hide yes)
@@
 			)
 		)
-		(property "Footprint" ""
+		(property "Footprint" "Package_SO:SOIC-8_3.9x4.9mm_P1.27mm"
 			(at 116.84 62.23 0)
 			(hide yes)
@@
 			)
 		)
-		(property "Footprint" ""
+		(property "Footprint" "Capacitor_SMD:C_0805_2012Metric"
 			(at 98.7552 58.42 0)
 			(hide yes)
@@
 			)
 		)
-		(property "Footprint" ""
+		(property "Footprint" "Resistor_SMD:R_0805_2012Metric"
 			(at 34.29 65.278 90)
 			(hide yes)
@@
 			)
 		)
-		(property "Footprint" ""
+		(property "Footprint" "Resistor_SMD:R_0805_2012Metric"
 			(at 87.122 49.53 90)
 			(hide yes)

Commit message: cleaned 3,4
Parts:
- removed R11: R, Resistor_SMD:R_0805_2012Metric, symbol Device:R
- added C7: 100n, Capacitor_SMD:C_01005_0402Metric, symbol Device:C
- C10: value C -> 1n
- C11, C9: value C -> 100n; footprint Capacitor_SMD:C_0805_2012Metric -> Capacitor_SMD:C_01005_0402Metric
- C5, C8: value C -> 100p
- R10, R7: value R -> 2k
Connections:
- net GND: now also C7.2; no longer C10.2, C11.2, D5.2 (A), D6.2 (A), U1.4 (V-), U1.5 (Ref)
- net VCC: now also C9.2; no longer U1.7 (V+)
- net at C5.1, D3.1 (K), R7.2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: now also C10.1, D4.2 (A); no longer D4.1 (K)
- new net: C7.1, U1.5 (Ref)
- new net: C10.2, D5.1 (K), D6.2 (A), U1.2 (-)
- new net: C9.1, U1.7 (V+)
- new net: C8.1, R10.2
- new net: C11.1, D5.2 (A), U1.4 (V-)
- new net +5V: D4.1 (K), D6.1 (K)
- new net -5V: C11.2, D3.2 (A)
- now unconnected: U1.1 (Rg), U1.8 (Rg)
- no-connect marks 0 -> 2
Other:
- note added: "100n capaacitors at pin7,4 are for decoupling"
- note added: "Diodes are for over voltage protection"
- note added: "both pin 3,2 have not been connected to input so that some differential input may exist"
- note added: "leave pin 1,8 as is or put Rg between them for a non unity gain"
- moved on the sheet: C10, D4, D6
