File: MCU/mcu/instrumentation_amplifier.kicad_sch (KiCad schematic)
At the start: 13 parts, among them U1 INA128

Commit message: changed
Parts:
- removed C7: 100n, Capacitor_SMD:C_01005_0402Metric, symbol Device:C
Connections:
- net VCC is gone; now on net +5V: C9.2
- net +5V: now also D4.2 (A), D6.2 (A), U1.7 (V+); no longer D4.1 (K), D6.1 (K)
- net -5V: now also C11.1, D3.1 (K), D5.1 (K), U1.4 (V-); no longer C11.2, D3.2 (A)
- net GND: now also C11.2, C9.1, U1.5 (Ref)
- net at C10.1, C5.1, R7.2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: now also D3.2 (A), D4.1 (K); no longer D3.1 (K), D4.2 (A)
- net at C10.2, U1.2 (-): now also C8.1, D5.2 (A), D6.1 (K), R10.2; no longer D5.1 (K), D6.2 (A)
- net In renamed In+
- net In+: no longer R10.1
- new net In-: R10.1
Other:
- note added: ".options compatibility=ps"
- moved on the sheet: D3, D4, D5, D6
