File: MCU/mcu/signal_conditioning.kicad_sch (KiCad schematic)
At the start: 5 parts, among them T1 SCT-013-000

Commit message: changed
Connections:
- net GND: now also D1.1 (A), R1.1, T1.4 (SB); no longer D1.2 (K)
- net Out: now also D1.3 (COM); no longer D1.1 (A), R1.1, T1.4 (SB)
- net VCC: now also D1.2 (K); no longer D1.3 (COM)
Changed lines of the file:
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@@
 	(paper "A4")
-	(junction
-		(at 76.2 53.34)
-		(diameter 0)
-		(color 0 0 0 0)
-	)
 	(junction
 		(at 33.02 92.71)
@@
 	)
 	(junction
-		(at 93.98 63.5)
+		(at 77.47 53.34)
 		(diameter 0)
 		(color 0 0 0 0)
 	)
 	(junction
-		(at 86.36 73.66)
+		(at 77.47 48.26)
+		(diameter 0)
+		(color 0 0 0 0)
+	)
+	(junction
+		(at 93.98 63.5)
 		(diameter 0)
 		(color 0 0 0 0)
@@
 		(color 0 0 0 0)
 	)
+	(junction
+		(at 78.74 54.61)
+		(diameter 0)
+		(color 0 0 0 0)
+	)
 	(wire
 		(pts
@@
 	(wire
 		(pts
-			(xy 86.36 73.66) (xy 86.36 77.47)
+			(xy 81.28 49.53) (xy 81.28 54.61)
+		)
+		(stroke
+			(width 0)
+			(type default)
+		)
+	)
+	(wire
+		(pts
+			(xy 81.28 54.61) (xy 78.74 54.61)
 		)
 		(stroke
@@
 	(wire
 		(pts
-			(xy 76.2 44.45) (xy 76.2 53.34)
-		)
-		(stroke
-			(width 0)
-			(type default)
-		)
-	)
-	(wire
-		(pts
 			(xy 71.12 53.34) (xy 71.12 54.61)
 		)
@@
 	(wire
 		(pts
+			(xy 77.47 48.26) (xy 77.47 53.34)
+		)
+		(stroke
+			(width 0)
+			(type default)
+		)
+	)
+	(wire
+		(pts
 			(xy 33.02 63.5) (xy 34.29 63.5)
 		)
@@
 	(wire
 		(pts
-			(xy 78.74 53.34) (xy 76.2 53.34)
+			(xy 77.47 53.34) (xy 78.74 53.34)
 		)
 		(stroke
@@
 	(wire
 		(pts
-			(xy 78.74 58.42) (xy 78.74 53.34)
-		)
-		(stroke
-			(width 0)
-			(type default)
-		)
-	)
-	(wire
-		(pts
-			(xy 71.12 53.34) (xy 76.2 53.34)
+			(xy 78.74 58.42) (xy 78.74 54.61)
+		)
+		(stroke
+			(width 0)
+			(type default)
+		)
+	)
+	(wire
+		(pts
+			(xy 71.12 53.34) (xy 77.47 53.34)
 		)
 		(stroke
@@
 	(wire
 		(pts
-			(xy 86.36 63.5) (xy 86.36 73.66)
+			(xy 78.74 54.61) (xy 78.74 53.34)
+		)
+		(stroke
+			(width 0)
+			(type default)
+		)
+	)
+	(wire
+		(pts
+			(xy 86.36 63.5) (xy 86.36 68.58)
+		)
+		(stroke
+			(width 0)
+			(type default)
+		)
+	)
+	(wire
+		(pts
+			(xy 77.47 46.99) (xy 77.47 48.26)
 		)
 		(stroke
@@
 		)
 	)
-	(wire
-		(pts
-			(xy 33.02 92.71) (xy 34.29 92.71)
-		)
-		(stroke
-			(width 0)
-			(type default)
+	(hierarchical_label "Out+"
+		(shape output)
+		(at 81.28 49.53 90)
+		(effects
+			(font
+				(size 1.27 1.27)
+			)
+			(justify left)
 		)
 	)
 	(hierarchical_label "Out"
 		(shape output)
-		(at 76.2 44.45 0)
+		(at 86.36 68.58 0)
 		(effects
 			(font
@@
 	(symbol
 		(lib_id "power:VCC")
-		(at 86.36 77.47 180)
+		(at 93.98 67.31 180)
 		(unit 1)
 		(body_style 1)
@@
 		(fields_autoplaced yes)
 		(property "Reference" "#PWR02"
-			(at 86.36 73.66 0)
+			(at 93.98 63.5 0)
 			(hide yes)
 			(show_name no)
@@
 		)
 		(property "Value" "VCC"
-			(at 86.36 82.55 0)
+			(at 93.98 72.39 0)
 			(show_name no)
 			(do_not_autoplace no)
@@
 		)
 		(property "Footprint" ""
-			(at 86.36 77.47 0)
+			(at 93.98 67.31 0)
 			(hide yes)
 			(show_name no)
@@
 		)
 		(property "Datasheet" ""
-			(at 86.36 77.47 0)
+			(at 93.98 67.31 0)
 			(hide yes)
 			(show_name no)
@@
 		)
 		(property "Description" "Power symbol creates a global label with name \"VCC\""
-			(at 86.36 77.47 0)
+			(at 93.98 67.31 0)
 			(hide yes)
 			(show_name no)
@@
 			)
 		)
-		(property "Sim.Params" "dc=0 ampl=0.2 f=25000 td=0 theta=0 phase=0 ac=1"
+		(property "Sim.Params" "dc=0 ampl=1 f=1k ac=1"
 			(at 36.83 90.0401 0)
 			(show_name no)
@@
 	(symbol
 		(lib_id "power:GND")
-		(at 93.98 67.31 0)
+		(at 77.47 46.99 180)
 		(unit 1)
 		(body_style 1)
@@
 		(fields_autoplaced yes)
 		(property "Reference" "#PWR01"
-			(at 93.98 73.66 0)
+			(at 77.47 40.64 0)
 			(hide yes)
 			(show_name no)
@@
 		)
 		(property "Value" "GND"
-			(at 93.98 72.39 0)
+			(at 77.47 41.91 0)
 			(show_name no)
 			(do_not_autoplace no)
@@
 		)
 		(property "Footprint" ""
-			(at 93.98 67.31 0)
+			(at 77.47 46.99 0)
 			(hide yes)
 			(show_name no)
@@
 		)
 		(property "Datasheet" ""
-			(at 93.98 67.31 0)
+			(at 77.47 46.99 0)
 			(hide yes)
 			(show_name no)
@@
 		)
 		(property "Description" "Power symbol creates a global label with name \"GND\" , ground"
-			(at 93.98 67.31 0)
+			(at 77.47 46.99 0)
 			(hide yes)
 			(show_name no)
@@
 				(path "/a05656f2-56dd-4122-820d-a34d3928231b/7a76ff6f-6805-4348-9ded-bfb68948d758"
 					(reference "#PWR01")
-					(unit 1)
-				)
-			)
-		)
-	)
-	(symbol
-		(lib_id "power:PWR_FLAG")
-		(at 86.36 73.66 90)
-		(unit 1)
-		(body_style 1)
-		(exclude_from_sim no)
-		(in_bom yes)
-		(on_board yes)
-		(in_pos_files yes)
-		(dnp no)
-		(property "Reference" "#FLG01"
-			(at 84.455 73.66 0)
-			(hide yes)
-			(show_name no)
-			(do_not_autoplace no)
-			(effects
-				(font
-					(size 1.27 1.27)
-				)
-			)
-		)
-		(property "Value" "PWR_FLAG"
-			(at 78.486 73.66 90)
-			(show_name no)
-			(do_not_autoplace no)
-			(effects
-				(font
-					(size 1.27 1.27)
-				)
-			)
-		)
-		(property "Footprint" ""
-			(at 86.36 73.66 0)
-			(hide yes)
-			(show_name no)
-			(do_not_autoplace no)
-			(effects
-				(font
-					(size 1.27 1.27)
-				)
-			)
-		)
-		(property "Datasheet" ""
-			(at 86.36 73.66 0)
-			(hide yes)
-			(show_name no)
-			(do_not_autoplace no)
-			(effects
-				(font
-					(size 1.27 1.27)
-				)
-			)
-		)
-		(property "Description" "Special symbol for telling ERC where power comes from"
-			(at 86.36 73.66 0)
-			(hide yes)
-			(show_name no)
-			(do_not_autoplace no)
-			(effects
-				(font
-					(size 1.27 1.27)
-				)
-			)
-		)
-		(pin "1"
-		)
-		(instances
-			(project "mcu"
-				(path "/a05656f2-56dd-4122-820d-a34d3928231b/7a76ff6f-6805-4348-9ded-bfb68948d758"
-					(reference "#FLG01")
 					(unit 1)
 				)
@@
 			)
 		)
-		(property "Sim.Params" "dc=1.65 ampl=1 f=60 td=0 theta=0 phase=0 ac=1 ph=0 portnum=0 z0=0.1"
+		(property "Sim.Params" "dc=0 ampl=1 f=1k ac=1"
 			(at 38.1 60.8301 0)
 			(show_name no)
@@
 					(unit 1)
 				)
+			)
+		)
+	)
+	(symbol
+		(lib_id "power:PWR_FLAG")
+		(at 77.47 48.26 90)
+		(unit 1)
+		(body_style 1)
+		(exclude_from_sim no)
+		(in_bom yes)
+		(on_board yes)
+		(in_pos_files yes)
+		(dnp no)
+		(property "Reference" "#FLG01"
+			(at 75.565 48.26 0)
+			(hide yes)
+			(show_name no)
+			(do_not_autoplace no)
+			(effects
+				(font
+					(size 1.27 1.27)
+				)
+			)
+		)
+		(property "Value" "PWR_FLAG"
+			(at 69.596 48.26 90)
+			(show_name no)
+			(do_not_autoplace no)
+			(effects
+				(font
+					(size 1.27 1.27)
+				)
+			)
+		)
+		(property "Footprint" ""
+			(at 77.47 48.26 0)
+			(hide yes)
+			(show_name no)
+			(do_not_autoplace no)
+			(effects
+				(font
+					(size 1.27 1.27)
+				)
+			)
+		)
+		(property "Datasheet" ""
+			(at 77.47 48.26 0)
+			(hide yes)
+			(show_name no)
+			(do_not_autoplace no)
+			(effects
+				(font
+					(size 1.27 1.27)
+				)
+			)
+		)
+		(property "Description" "Special symbol for telling ERC where power comes from"
+			(at 77.47 48.26 0)
+			(hide yes)
+			(show_name no)
+			(do_not_autoplace no)
+			(effects
+				(font
+					(size 1.27 1.27)
+				)
+			)
+		)
+		(pin "1"
+		)
+		(instances
+			(project "mcu"
+				(path "/a05656f2-56dd-4122-820d-a34d3928231b/7a76ff6f-6805-4348-9ded-bfb68948d758"
+					(reference "#FLG01")
+					(unit 1)
+				)
