File: MCU/mcu/mcu.kicad_sch (KiCad schematic)
At the start: 0 parts

Commit message: worked on unit 5
Other:
- sheet output clamp and ADC Interface ports: added In; removed none
Changed lines of the file:
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@@
+	(wire
+		(pts
+			(xy 74.93 44.45) (xy 74.93 46.99)
+		)
+		(stroke
+			(width 0)
+			(type default)
+		)
+	)
+	(wire
+		(pts
+			(xy 87.63 44.45) (xy 74.93 44.45)
+		)
+		(stroke
+			(width 0)
+			(type default)
+		)
+	)
 	(wire
 		(pts
 			(xy 177.8 45.72) (xy 179.07 45.72)
+		)
+		(stroke
+			(width 0)
+			(type default)
+		)
+	)
+	(wire
+		(pts
+			(xy 74.93 46.99) (xy 67.31 46.99)
 		)
 		(stroke
@@
 			)
 		)
+		(pin "In" input
+			(at 67.31 46.99 0)
+			(effects
+				(font
+					(size 1.27 1.27)
+				)
+				(justify right)
+			)
+		)
