File: MCU/mcu/mcu.kicad_sch (KiCad schematic)
At the start: 0 parts

Commit message: changed
Other:
- removed sheet DC_Bias
- sheet instrumentation_amplifier ports: added In+, In-; removed In
- sheet signal_conditioning ports: added Out+; removed none
Changed lines of the file:
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@@
 	(generator_version "10.0")
 	(paper "A4")
-	(junction
-		(at 177.8 45.72)
-		(diameter 0)
-		(color 0 0 0 0)
-	)
-	(wire
-		(pts
-			(xy 167.64 45.72) (xy 177.8 45.72)
-		)
-		(stroke
-			(width 0)
-			(type default)
-		)
-	)
-	(wire
-		(pts
-			(xy 137.16 45.72) (xy 149.86 45.72)
+	(wire
+		(pts
+			(xy 187.96 45.72) (xy 187.96 31.75)
+		)
+		(stroke
+			(width 0)
+			(type default)
+		)
+	)
+	(wire
+		(pts
+			(xy 167.64 50.8) (xy 175.26 50.8)
+		)
+		(stroke
+			(width 0)
+			(type default)
+		)
+	)
+	(wire
+		(pts
+			(xy 187.96 31.75) (xy 156.21 31.75)
+		)
+		(stroke
+			(width 0)
+			(type default)
+		)
+	)
+	(wire
+		(pts
+			(xy 175.26 53.34) (xy 175.26 50.8)
+		)
+		(stroke
+			(width 0)
+			(type default)
+		)
+	)
+	(wire
+		(pts
+			(xy 156.21 31.75) (xy 156.21 36.83)
+		)
+		(stroke
+			(width 0)
+			(type default)
+		)
+	)
+	(wire
+		(pts
+			(xy 210.82 53.34) (xy 175.26 53.34)
 		)
 		(stroke
@@
 	(wire
 		(pts
-			(xy 177.8 45.72) (xy 179.07 45.72)
-		)
-		(stroke
-			(width 0)
-			(type default)
-		)
-	)
-	(wire
-		(pts
 			(xy 74.93 46.99) (xy 67.31 46.99)
 		)
@@
 	(wire
 		(pts
-			(xy 190.5 45.72) (xy 207.01 45.72)
-		)
-		(stroke
-			(width 0)
-			(type default)
-		)
-	)
-	(netclass_flag ""
-		(length 2.54)
-		(shape round)
-		(at 48.26 95.25 0)
+			(xy 187.96 45.72) (xy 205.74 45.72)
+		)
+		(stroke
+			(width 0)
+			(type default)
+		)
+	)
+	(wire
+		(pts
+			(xy 205.74 44.45) (xy 205.74 45.72)
+		)
+		(stroke
+			(width 0)
+			(type default)
+		)
+	)
+	(wire
+		(pts
+			(xy 205.74 44.45) (xy 210.82 44.45)
+		)
+		(stroke
+			(width 0)
+			(type default)
+		)
+	)
+	(wire
+		(pts
+			(xy 105.41 44.45) (xy 118.11 44.45)
+		)
+		(stroke
+			(width 0)
+			(type default)
+		)
+	)
+	(sheet
+		(at 87.63 41.91)
+		(size 17.78 3.81)
+		(exclude_from_sim no)
+		(in_bom yes)
+		(on_board yes)
+		(dnp no)
 		(fields_autoplaced yes)
-		(effects
-			(font
-				(size 1.27 1.27)
-			)
-			(justify left bottom)
-		)
-		(property "Netclass" ".tran 0 100m"
-			(at 48.9585 92.71 0)
-			(show_name no)
-			(do_not_autoplace no)
+		(stroke
+			(width 0.1524)
+			(type solid)
+		)
+		(fill
+			(color 0 0 0 0)
+		)
+		(property "Sheetname" "anti_aliasing"
+			(at 87.63 41.1984 0)
+			(show_name no)
+			(do_not_autoplace no)
+			(effects
+				(font
+					(size 1.27 1.27)
+				)
+				(justify left bottom)
+			)
+		)
+		(property "Sheetfile" "anti_aliasing.kicad_sch"
+			(at 87.63 46.3046 0)
+			(show_name no)
+			(do_not_autoplace no)
+			(effects
+				(font
+					(size 1.27 1.27)
+				)
+				(justify left top)
+			)
+		)
+		(pin "In" input
+			(at 105.41 44.45 0)
+			(effects
+				(font
+					(size 1.27 1.27)
+				)
+				(justify right)
+			)
+		)
+		(pin "Out" output
+			(at 87.63 44.45 180)
 			(effects
 				(font
@@
 			)
 		)
-		(property "Component Class" ""
-			(at 119.38 53.34 0)
-			(show_name no)
-			(do_not_autoplace no)
-			(effects
-				(font
-					(size 1.27 1.27)
-					(italic yes)
+		(instances
+			(project "mcu"
+				(path "/a05656f2-56dd-4122-820d-a34d3928231b"
+					(page "4")
 				)
 			)
@@
 	)
 	(sheet
-		(at 87.63 36.83)
+		(at 118.11 36.83)
 		(size 49.53 17.78)
 		(exclude_from_sim no)
@@
 		)
 		(property "Sheetname" "instrumentation_amplifier"
-			(at 87.63 36.1184 0)
+			(at 118.11 36.1184 0)
 			(show_name no)
 			(do_not_autoplace no)
@@
 		)
 		(property "Sheetfile" "instrumentation_amplifier.kicad_sch"
-			(at 87.63 55.1946 0)
+			(at 118.11 55.1946 0)
 			(show_name no)
 			(do_not_autoplace no)
@@
 			)
 		)
-		(pin "In" output
-			(at 137.16 45.72 0)
+		(pin "Out" output
+			(at 118.11 44.45 180)
+			(effects
+				(font
+					(size 1.27 1.27)
+				)
+				(justify left)
+			)
+		)
+		(pin "In+" input
+			(at 156.21 36.83 90)
 			(effects
 				(font
@@
 			)
 		)
-		(pin "Out" output
-			(at 87.63 44.45 180)
-			(effects
-				(font
-					(size 1.27 1.27)
-				)
-				(justify left)
+		(pin "In-" input
+			(at 167.64 50.8 0)
+			(effects
+				(font
+					(size 1.27 1.27)
+				)
+				(justify right)
 			)
 		)
@@
 	)
 	(sheet
-		(at 177.8 43.18)
-		(size 12.7 3.81)
+		(at 210.82 41.91)
+		(size 34.29 16.51)
 		(exclude_from_sim no)
 		(in_bom yes)
@@
 			(color 0 0 0 0)
 		)
-		(property "Sheetname" "DC_Bias"
-			(at 177.8 42.4684 0)
+		(property "Sheetname" "signal_conditioning"
+			(at 210.82 41.1984 0)
 			(show_name no)
 			(do_not_autoplace no)
@@
 			)
 		)
-		(property "Sheetfile" "DC_Bias.kicad_sch"
-			(at 177.8 47.5746 0)
+		(property "Sheetfile" "signal_conditioning.kicad_sch"
+			(at 210.82 59.0046 0)
 			(show_name no)
 			(do_not_autoplace no)
@@
 			)
 		)
-		(pin "In" input
-			(at 190.5 45.72 0)
-			(effects
-				(font
-					(size 1.27 1.27)
-				)
-				(justify right)
-			)
-		)
 		(pin "Out" output
-			(at 177.8 45.72 180)
+			(at 210.82 44.45 180)
 			(effects
 				(font
@@
 			)
 		)
-		(instances
-			(project "mcu"
-				(path "/a05656f2-56dd-4122-820d-a34d3928231b"
-					(page "3")
-				)
-			)
-		)
-	)
-	(sheet
-		(at 207.01 43.18)
-		(size 12.7 3.81)
-		(exclude_from_sim no)
-		(in_bom yes)
-		(on_board yes)
-		(dnp no)
-		(fields_autoplaced yes)
-		(stroke
-			(width 0.1524)
-			(type solid)
-		)
-		(fill
-			(color 0 0 0 0)
-		)
-		(property "Sheetname" "signal_conditioning"
-			(at 207.01 42.4684 0)
-			(show_name no)
-			(do_not_autoplace no)
-			(effects
-				(font
-					(size 1.27 1.27)
-				)
-				(justify left bottom)
-			)
-		)
-		(property "Sheetfile" "signal_conditioning.kicad_sch"
-			(at 207.01 47.5746 0)
-			(show_name no)
-			(do_not_autoplace no)
-			(effects
-				(font
-					(size 1.27 1.27)
-				)
-				(justify left top)
-			)
-		)
-		(pin "Out" output
-			(at 207.01 45.72 180)
+		(pin "Out+" output
+			(at 210.82 53.34 180)
 			(effects
 				(font
@@
 				)
 			)
-		)
-	)
-	(sheet
-		(at 149.86 43.18)
-		(size 17.78 3.81)
-		(exclude_from_sim no)
-		(in_bom yes)
-		(on_board yes)
-		(dnp no)
-		(fields_autoplaced yes)
-		(stroke
-			(width 0.1524)
-			(type solid)
-		)
-		(fill
-			(color 0 0 0 0)
-		)
-		(property "Sheetname" "anti_aliasing"
-			(at 149.86 42.4684 0)
-			(show_name no)
-			(do_not_autoplace no)
-			(effects
-				(font
-					(size 1.27 1.27)
-				)
-				(justify left bottom)
-			)
-		)
-		(property "Sheetfile" "anti_aliasing.kicad_sch"
-			(at 149.86 47.5746 0)
-			(show_name no)
-			(do_not_autoplace no)
-			(effects
-				(font
-					(size 1.27 1.27)
-				)
-				(justify left top)
-			)
-		)
-		(pin "In" input
-			(at 167.64 45.72 0)
-			(effects
-				(font
-					(size 1.27 1.27)
-				)
-				(justify right)
-			)
-		)
-		(pin "Out" output
-			(at 149.86 45.72 180)
-			(effects
-				(font
-					(size 1.27 1.27)
-				)
-				(justify left)
-			)
-		)
-		(instances
-			(project "mcu"
-				(path "/a05656f2-56dd-4122-820d-a34d3928231b"
-					(page "4")
-				)
-			)

Commit message: yy
Other:
- added sheet test (test.kicad_sch)
Changed lines of the file:
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@@
+	)
+	(sheet
+		(at 66.04 92.71)
+		(size 12.7 6.35)
+		(exclude_from_sim no)
+		(in_bom yes)
+		(on_board yes)
+		(dnp no)
+		(fields_autoplaced yes)
+		(stroke
+			(width 0.1524)
+			(type solid)
+		)
+		(fill
+			(color 0 0 0 0)
+		)
+		(property "Sheetname" "test"
+			(at 66.04 91.9984 0)
+			(show_name no)
+			(do_not_autoplace no)
+			(effects
+				(font
+					(size 1.27 1.27)
+				)
+				(justify left bottom)
+			)
+		)
+		(property "Sheetfile" "test.kicad_sch"
+			(at 66.04 99.6446 0)
+			(show_name no)
+			(do_not_autoplace no)
+			(effects
+				(font
+					(size 1.27 1.27)
+				)
+				(justify left top)
+			)
+		)
+		(instances
+			(project "mcu"
+				(path "/a05656f2-56dd-4122-820d-a34d3928231b"
+					(page "3")
+				)
+			)
+		)
 	)
 	(sheet
