File: MCU/mcu/test.kicad_sch (KiCad schematic)
At the start: 12 parts, among them U1 INA128

Commit message: yy
Parts:
- removed C10: 1n, Capacitor_SMD:C_0805_2012Metric, symbol Device:C
- removed C11, C9: 100n, Capacitor_SMD:C_01005_0402Metric, symbol Device:C
- removed C5, C8: 100p, Capacitor_SMD:C_0805_2012Metric, symbol Device:C
- removed D3, D4, D5, D6: 1N4148, Diode_THT:D_DO-35_SOD27_P7.62mm_Horizontal, symbol Diode:1N4148
- removed R10, R7: 2k, Resistor_SMD:R_0805_2012Metric, symbol Device:R
- removed U1: INA128, Package_SO:SOIC-8_3.9x4.9mm_P1.27mm, symbol Amplifier_Instrumentation:INA128
- added C15: 360p, Capacitor_SMD:C_0805_2012Metric, symbol Device:C
- added C17: 150p, symbol Device:C
- added C3: 1n, symbol Device:C
- added C7: 430pf, Capacitor_SMD:C_0805_2012Metric, symbol Device:C
- added R11, R8: 20k, Resistor_SMD:R_0805_2012Metric, symbol Device:R
- added R14, R4: 20k, symbol Device:R
- added U5: MCP6002-xMS, Package_SO:MSOP-8_3x3mm_P0.65mm, symbol Amplifier_Operational:MCP6002-xMS
- added V6: VSIN, symbol Simulation_SPICE:VSIN
Connections:
- net +5V: now also C15.1, C17.2, U5.4 (V-), U5.8 (V+), V6.2
- net Out: now also C3.1, U5.6 (-), U5.7
- new net: C15.2, R11.2, U5.3 (+)
- new net: C7.2, R4.1, U5.1, U5.2 (-)
- new net: C17.1, R14.2, U5.5 (+)
- new net: C3.2, R14.1, R4.2
- new net: C7.1, R11.1, R8.2
- new net: R8.1, V6.1
- no-connect marks 2 -> 0
Other:
- note added: ".ac dec 20 1 1Meg"
- note removed: ".options compatibility=all"
- note removed: "100n capaacitors at pin7,4 are for decoupling"
- note removed: "Diodes are for over voltage protection"
- note removed: "both pin 3,2 have not been connected to input so that some differential input may exist"
- note removed: "leave pin 1,8 as is or put Rg between them for a non unity gain"
