File: STM32/STM32.kicad_sch (KiCad schematic)
At the start: 6 parts, among them U1 STM32F103C8Tx

Commit message: completed stm32 phils lab video project schematic
Parts:
- added C10, C11: 10p, Capacitor_SMD:C_0402_1005Metric, symbol Device:C
- added C12: 23u, Capacitor_SMD:C_0402_1005Metric, symbol Device:C
- added C13: 22u, Capacitor_SMD:C_0402_1005Metric, symbol Device:C
- added C6: 10n, Capacitor_SMD:C_0402_1005Metric, symbol Device:C
- added C7: 1u, Capacitor_SMD:C_0402_1005Metric, symbol Device:C
- added C8: C, Capacitor_SMD:C_0402_1005Metric, symbol Device:C
- added C9: 100n, Capacitor_SMD:C_0402_1005Metric, symbol Device:C
- added D1: LED, LED_SMD:LED_0201_0603Metric, symbol Device:LED
- added FB1: 120R, Inductor_SMD:L_0402_1005Metric, symbol Device:FerriteBead
- added J1: USB_B_Micro, Connector_USB:USB_Micro-B_Wuerth_614105150721_Vertical, symbol Connector:USB_B_Micro
- added J2, J3, J4: Conn_01x04_Pin, Connector_PinHeader_2.54mm:PinHeader_1x04_P2.54mm_Vertical, symbol Connector:Conn_01x04_Pin
- added R1: 10k, Resistor_SMD:R_0402_1005Metric, symbol Device:R
- added R2, R3, R4, R6: 1.5k, Resistor_SMD:R_0402_1005Metric, symbol Device:R
- added SW1: SW_SPDT, Button_Switch_THT:SW_E-Switch_EG1224_SPDT_Angled, symbol Switch:SW_SPDT
- added U2: AMS1117-3.3, Package_TO_SOT_SMD:SOT-223-3_TabPin2, symbol Regulator_Linear:AMS1117-3.3
- added Y1: Crystal_GND24, Crystal:Crystal_SMD_3225-4Pin_3.2x2.5mm, symbol Device:Crystal_GND24
- C1, C2, C3, C4, C5: footprint (none) -> Capacitor_SMD:C_0402_1005Metric
Connections:
- net +3.3V: now also C13.1, C8.1, D1.2 (A), FB1.2, J2.1 (Pin_1), J3.1 (Pin_1), J4.1 (Pin_1), R2.1, R4.1, R6.1, SW1.3 (C), U2.2 (VO)
- net GND: now also C10.2, C11.1, C12.2, C13.2, C6.2, C7.2, C8.2, C9.2, J1.5 (GND), J2.4 (Pin_4), J3.4 (Pin_4), J4.4 (Pin_4), R3.2, SW1.1 (A), U2.1 (GND), Y1.2 (G), Y1.4 (G)
- net I2C2_SC1: now reaches U1.21 (PB10)
- net I2C2_SC1: now also J4.2 (Pin_2), R4.2
- net I2C2_SDA: now reaches U1.22 (PB11)
- net I2C2_SDA: now also J4.3 (Pin_3), R6.2
- net USB_D-: now reaches U1.32 (PA11)
- net USB_D-: now also J1.2 (D-), R2.2
- net USB_D+: now reaches U1.33 (PA12)
- net USB_D+: now also J1.3 (D+)
- net SWDIO: now reaches U1.34 (PA13)
- net SWDIO: now also J2.2 (Pin_2)
- net SWCLK: now reaches U1.37 (PA14)
- net SWCLK: now also J2.3 (Pin_3)
- net USART_TX: now reaches U1.42 (PB6)
- net USART_TX: now also J3.2 (Pin_2)
- net USART_RX: now reaches U1.43 (PB7)
- net USART_RX: now also J3.3 (Pin_3)
- net at U1.44 (BOOT0): now also R1.1
- net HSE_IN: now reaches U1.5 (PD0)
- net HSE_IN: now also C11.2, Y1.1
- net HSE_OUT: now reaches U1.6 (PD1)
- net HSE_OUT: now also C10.1, Y1.3
- net NRST: now reaches U1.7 (NRST)
- net NRST: now also C9.1
- net +3.3VA: now reaches U1.9 (VDDA)
- net +3.3VA: now also C6.1, C7.1, FB1.1
- new net: R1.2, SW1.2 (B)
- new net PWR_LED_K: D1.1 (K), R3.1
- new net VBUS: C12.1, J1.1 (VBUS), U2.3 (VI)
- no-connect marks 0 -> 29
Other:
- note added: "10 MHz Crystal"
- note added: "3.3V is for digital systems and 3.3VA is for analog systems"
- note added: "Add NRST pin label so it's easier to handle during simulations and PCB routing"
- note added: "Not connecting USB Shield"
- note added: "Using the STM and Oscillator official Documentation, we find the right connections"
- note added: "digital to analog rail link"
- note added: "ferrite bead acts as a speed bump to unwanted energy spikes, absorbing them and then releasing them as heat"
- moved on the sheet: C1, C2, C3, C4, C5, U1
