File: MCU/test/test.kicad_sch (KiCad schematic)
At the start: 0 parts

Commit message: hh
Parts:
- added C1: 330p, symbol Device:C
- added C2: 150p, symbol Device:C
- added C4: 430pf, Capacitor_SMD:C_0805_2012Metric, symbol Device:C
- added C6: 360p, Capacitor_SMD:C_0805_2012Metric, symbol Device:C
- added R2, R3: 20k, symbol Device:R
- added R5, R6: 20k, Resistor_SMD:R_0805_2012Metric, symbol Device:R
- added U2: MCP6002-xMS, Package_SO:MSOP-8_3x3mm_P0.65mm, symbol Amplifier_Operational:MCP6002-xMS
- added V1: 5, symbol Simulation_SPICE:VDC
- added V3, V4: VSIN, symbol Simulation_SPICE:VSIN
Connections:
- new net: R5.1, V4.1
- new net: C4.1, R5.2, R6.1
- new net: C4.2, R3.1, U2.1, U2.2 (-)
- new net: C6.2, R6.2, U2.3 (+)
- new net: C2.1, R2.2, U2.5 (+)
- new net: V3.1, V4.2
- new net: U2.8 (V+), V1.1
- new net: C1.2, R2.1, R3.2
- new net GND: C2.2, C6.1, U2.4 (V-), V1.2, V3.2
- new net Out: C1.1, U2.6 (-), U2.7
Other:
- note added: ".ac dec 20 1 1Meg"

Commit message: k
fitrst test folder
Parts:
- removed U2: MCP6002-xMS, Package_SO:MSOP-8_3x3mm_P0.65mm, symbol Amplifier_Operational:MCP6002-xMS
- added U1: OPA2197xD, Package_SO:SOIC-8_3.9x4.9mm_P1.27mm, symbol Amplifier_Operational:OPA2197xD
- C1: value 330p -> 33n
- C2: value 150p -> 10n
- C4: value 430pf -> 3.6n
- C6: value 360p -> 9.6n
- R2, R3, R5, R6: value 20k -> 6.34k
Connections:
- net GND: now also U1.4 (V-)
- net Out: now also U1.6 (-), U1.7
- net at R5.2, R6.1: now also C6.2; no longer C4.1
- net at C4.2, R3.1: now also U1.1, U1.2 (-)
- net at R6.2: now also C4.1, U1.3 (+); no longer C6.2
- net at R2.2: now also C1.2, U1.5 (+); no longer C2.1
- net at V1.1: now also U1.8 (V+)
- net at R2.1, R3.2: now also C2.1; no longer C1.2

Commit message: jk
Parts:
- removed V4: VSIN, symbol Simulation_SPICE:VSIN
- added V2: 5, symbol Simulation_SPICE:VDC
- C1: value 33n -> 1n
- C2: value 10n -> 750p
- C4: value 3.6n -> 1n
- C6: value 9.6n -> 100p
- R2: value 6.34k -> 107k
- R3: value 6.34k -> 49.6k
- R5: value 6.34k -> 104k
- R6: value 6.34k -> 383k
Connections:
- net GND: now also V2.2; no longer U1.4 (V-)
- net at R5.1: now also V3.1
- net at R5.2, R6.1: now also C4.1; no longer C6.2
- net at R6.2, U1.3 (+): now also C6.2; no longer C4.1
- net at R2.2, U1.5 (+): now also C2.1; no longer C1.2
- net at R2.1, R3.2: now also C1.2; no longer C2.1
- new net: U1.4 (V-), V2.1

Commit message: simulated the filter
Parts:
- removed U1: OPA2197xD, Package_SO:SOIC-8_3.9x4.9mm_P1.27mm, symbol Amplifier_Operational:OPA2197xD
- added U2: LT6237, symbol Amplifier_Operational:LT6237
- R2: value 107k -> 105k
- R3: value 49.6k -> 51.1k
Connections:
- net GND: now also V2.1; no longer V2.2
- net Out: now also U2.6 (-), U2.7
- net at C4.2, R3.1: now also U2.1, U2.2 (-)
- net at V1.1: now also U2.8 (V+)
- net at C6.2, R6.2: now also U2.3 (+)
- net at C2.1, R2.2: now also U2.5 (+)
- new net: U2.4 (V-), V2.2
Other:
- moved on the sheet: V2
